File: poc/qclock.kicad_sch (KiCad schematic)
At the start: 39 parts, among them J1 Conn_01x04_Male, J2 Conn_01x04_Male, J3 USB_B_Micro, J4 Conn_01x04_Male, J5 Conn_01x03_Male, SW1 SW_SPDT, SW2 SW_Push, SW3 SW_Push, SW4 SW_Push, U1 STM32F103C8Tx, U2 AMS1117-3.3, Y1 Crystal_GND24

Commit message: Finish poc design
Parts:
- added H1, H2, H3, H4: MountingHole, MountingHole:MountingHole_2.2mm_M2, symbol Mechanical:MountingHole
