File: poc/_autosave-qclock.kicad_sch (KiCad schematic)
At the start: 43 parts, among them J1 Conn_01x04_Male, J2 Conn_01x04_Male, J3 USB_B_Micro, J4 Conn_01x04_Male, J5 Conn_01x03_Male, SW1 SW_SPDT, SW2 SW_Push, SW3 SW_Push, SW4 SW_Push, U1 STM32F103C8Tx, U2 AMS1117-3.3, Y1 Crystal_GND24

Commit message: Update
Parts:
- D1: footprint LED_SMD:LED_0402_1005Metric -> LED_SMD:LED_0603_1608Metric; JLCPCB Part #（optional） (none) -> C2290
- D2, D4: JLCPCB Part #（optional） (none) -> C2846931
- J3: JLCPCB Part #（optional） (none) -> C879727
- R1, R2, R3, R4: JLCPCB Part #（optional） (none) -> C25744
- SW1: footprint Button_Switch_SMD:SW_SPDT_PCM12 -> Button_Switch_SMD:SW_DIP_SPSTx01_Slide_6.7x4.1mm_W6.73mm_P2.54mm_LowProfile_JPin
- Y1: footprint Crystal:Crystal_SMD_0603-4Pin_6.0x3.5mm -> Crystal:Crystal_SMD_3225-4Pin_3.2x2.5mm
Changed lines of the file:
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@@
 			)
 		)
-		(property "Footprint" "Button_Switch_SMD:SW_SPDT_PCM12"
+		(property "Footprint" "Button_Switch_SMD:SW_DIP_SPSTx01_Slide_6.7x4.1mm_W6.73mm_P2.54mm_LowProfile_JPin"
 			(at 40.64 71.12 0)
 			(effects
@@
 			)
 		)
-		(property "JLCPCB Part #（optional）" ""
+		(property "JLCPCB Part #（optional）" " C25744"
 			(at 52.07 71.12 0)
 			(effects
@@
 			)
 		)
-		(property "Footprint" "Crystal:Crystal_SMD_0603-4Pin_6.0x3.5mm"
+		(property "Footprint" "Crystal:Crystal_SMD_3225-4Pin_3.2x2.5mm"
 			(at 45.72 92.71 0)
 			(effects
@@
 			)
 		)
-		(property "JLCPCB Part #（optional）" ""
+		(property "JLCPCB Part #（optional）" " C879727"
 			(at 166.37 115.57 0)
 			(effects
@@
 			)
 		)
-		(property "Footprint" "LED_SMD:LED_0402_1005Metric"
+		(property "Footprint" "LED_SMD:LED_0603_1608Metric"
 			(at 193.04 62.23 0)
 			(effects
@@
 			)
 		)
-		(property "JLCPCB Part #（optional）" ""
+		(property "JLCPCB Part #（optional）" "C2290"
 			(at 193.04 62.23 0)
 			(effects
@@
 			)
 		)
-		(property "JLCPCB Part #（optional）" ""
+		(property "JLCPCB Part #（optional）" " C25744"
 			(at 60.96 139.7 0)
 			(effects
@@
 			)
 		)
-		(property "JLCPCB Part #（optional）" ""
+		(property "JLCPCB Part #（optional）" " C25744"
 			(at 60.96 160.02 0)
 			(effects
@@
 			)
 		)
-		(property "JLCPCB Part #（optional）" ""
+		(property "JLCPCB Part #（optional）" " C25744"
 			(at 60.96 181.61 0)
 			(effects
@@
 			)
 		)
-		(property "JLCPCB Part #（optional）" ""
+		(property "JLCPCB Part #（optional）" "C2846931"
 			(at 252.73 87.63 0)
 			(effects
@@
 			)
 		)
-		(property "JLCPCB Part #（optional）" ""
+		(property "JLCPCB Part #（optional）" "C2846931"
 			(at 223.52 87.63 0)
 			(effects
