File: poc/qclock.kicad_pcb (KiCad board)
At the start: 2 copper layers, 39 parts, among them J1 Conn_01x04_Male, J2 Conn_01x04_Male, J3 USB_B_Micro, J4 Conn_01x04_Male, J5 Conn_01x03_Male, SW1 SW_SPDT, SW2 SW_Push, SW3 SW_Push, SW4 SW_Push, U1 STM32F103C8Tx, U2 AMS1117-3.3, Y1 Crystal_GND24

Commit message: Finish poc design
Parts:
- added H1: MountingHole, MountingHole:MountingHole_2.2mm_M2, F.Cu at (170.8, 100.0)
- added H2: MountingHole, MountingHole:MountingHole_2.2mm_M2, F.Cu at (170.8, 72.0)
- added H3: MountingHole, MountingHole:MountingHole_2.2mm_M2, F.Cu at (115.5, 72.0)
- added H4: MountingHole, MountingHole:MountingHole_2.2mm_M2, F.Cu at (115.5, 100.0)
- moved R1 79.8 mm to (156.2, 79.8)
- moved R5 77.0 mm to (160.0, 85.5), turned to 90 degrees
- moved R4 76.6 mm to (134.8, 74.3), turned to -90 degrees
- moved R3 68.3 mm to (134.8, 80.8), turned to -90 degrees
- moved C5 66.4 mm to (147.0, 81.8), turned to 90 degrees
- moved C4 65.8 mm to (158.0, 85.0), turned to -90 degrees
- moved C8 64.9 mm to (149.0, 81.0)
- moved Hour 63.9 mm to (132.0, 93.5)
- moved C14 62.1 mm to (120.3, 82.3), turned to -90 degrees
- moved R6 61.9 mm to (158.0, 96.2), turned to 90 degrees
- moved R2 61.1 mm to (135.0, 93.0), turned to 90 degrees
- moved C3 61.0 mm to (145.8, 83.0), turned to 90 degrees
- moved FB1 61.0 mm to (144.8, 93.0), turned to 180 degrees
- moved R8 60.7 mm to (150.5, 97.2)
- moved C2 60.4 mm to (149.0, 79.2)
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- renumbered SW2 to Hour, J4 to I2C, J5 to LED, SW3 to Minute, J2 to SWD, SW4 to Subminute, J1 to UART
Routing:
- net +3V3: track 0.00 -> 184.4 mm, vias 0 -> 9
- net VBUS: track 0.00 -> 104.6 mm, vias 0 -> 2
- net GND: track 0.00 -> 62.2 mm, vias 0 -> 32
- net /BTN_SM: track 0.00 -> 54.3 mm, vias 0 -> 2
- net /BTN_M: track 0.00 -> 50.7 mm, vias 0 -> 2
- net /LED: track 0.00 -> 44.7 mm, vias 0 -> 2
- net /BTN_H: track 0.00 -> 41.6 mm, vias 0 -> 2
- net Net-(SW1-B): track 0.00 -> 26.1 mm
- net /UART_RX: track 0.00 -> 25.1 mm, vias 0 -> 2
- net /UART_TX: track 0.00 -> 23.5 mm, vias 0 -> 2
- net /SWDIO: track 0.00 -> 18.2 mm
- net /SWCLK: track 0.00 -> 13.9 mm
- net /USB_D-: track 0.00 -> 12.5 mm
- net /USB_D+: track 0.00 -> 12.4 mm
- net /I2C2_SCL: track 0.00 -> 11.7 mm
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- added copper zone on F.Cu, net +3V3
- added copper zone on B.Cu, net GND
- added copper zone on F.Cu, net VBUS
Other:
- board outline added: 61.2 x 34 mm
- board text added: "Markus Glau 17.05.2024 QCLOCK controller"

Commit message: Redo files
Parts:
- renumbered UART to J1, SWD to J2, I2C to J4, LED to J5, Hour to SW2, Minute to SW3, Subminute to SW4
Other:
- board text added: "3v3 SCL SDA GND"
- board text added: "5V"
- board text added: "GND CLK DIO 3v3"
- board text added: "GND RX TX 3v3"
- board text added: "H"
- board text added: "L"
- board text added: "M"
- board text added: "SM"

Commit message: Update
Parts:
- D1: footprint LED_SMD:LED_0402_1005Metric -> LED_SMD:LED_0603_1608Metric
- SW1: footprint Button_Switch_SMD:SW_SPDT_PCM12 -> Button_Switch_SMD:SW_DIP_SPSTx01_Slide_6.7x4.1mm_W6.73mm_P2.54mm_LowProfile_JPin
- Y1: footprint Crystal:Crystal_SMD_0603-4Pin_6.0x3.5mm -> Crystal:Crystal_SMD_3225-4Pin_3.2x2.5mm
- moved Y1 1.48 mm to (140.0, 87.0)
- moved J1 0.88 mm to (144.6, 72.2)
- moved SW1 0.85 mm to (151.4, 72.0), turned to 0 degrees
- moved R4 0.78 mm to (134.5, 75.0)
Routing:
- net Net-(SW1-B): track 26.1 -> 18.5 mm
- net GND: track 62.2 -> 65.5 mm
- net +3V3: track 184.4 -> 183.3 mm
- net /HSE_OUT: track 11.5 -> 12.6 mm

Commit message: Final models
Parts:
- SW1: footprint Button_Switch_SMD:SW_DIP_SPSTx01_Slide_6.7x4.1mm_W6.73mm_P2.54mm_LowProfile_JPin -> footprints:CUS-12TB_NDC
- SW2, SW3, SW4: footprint Button_Switch_THT:SW_PUSH_6mm_H4.3mm -> btns:mybtn_smd
- moved SW2 4.37 mm to (128.2, 91.2), turned to 0 degrees
- moved SW3 3.40 mm to (128.2, 82.5)
- moved SW4 3.26 mm to (128.2, 73.8)
- moved SW1 0.84 mm to (151.8, 71.2), turned to 180 degrees
Routing:
- net +3V3: track 183.3 -> 192.9 mm
- net /BTN_H: track 41.6 -> 47.5 mm
- net Net-(SW1-B): track 18.5 -> 23.7 mm
- net GND: track 65.5 -> 63.6 mm, vias 32 -> 30
- net /BTN_SM: track 54.3 -> 56.1 mm
- net /BTN_M: track 50.7 -> 52.1 mm
