File: kicad/qclock.kicad_pcb (KiCad board)
At the start: 2 copper layers, 375 x 375 mm, 258 parts, among them J3 USB_B_Micro, U1 STM32F103C8Tx, U2 AMS1117-3.3, Y1 Crystal_GND24

Commit message: Final models
Parts:
- removed BOOT: SW_SPDT, Button_Switch_THT:SW_E-Switch_EG1271_DPDT
- removed C111, C112, C113, C114, C115, C116, C117, C118, C119, C120, C121, C122, C123, C14: 220n, Capacitor_SMD:C_0402_1005Metric
- removed D111: SK6805, LED_SMD:LED_SK6805_PLCC4_2.4x2.7mm_P1.3mm
- removed FB1: 120R, Inductor_SMD:L_0603_1608Metric
- removed HOUR, MINUTE, SUBMINUTE: SW_Push, Button_Switch_THT:SW_PUSH-12mm
- removed I2C: Conn_01x04_Male, Connector_PinSocket_2.54mm:PinSocket_1x04_P2.54mm_Horizontal
- removed J3: USB_B_Micro, Connector_USB:USB_Micro-B_Wuerth_629105150521
- removed R1, R2, R3, R4: 10k, Resistor_SMD:R_0402_1005Metric
- removed R5, R6, R7, R8: 1k5, Resistor_SMD:R_0402_1005Metric
- removed SWD, UART: Conn_01x04_Male, Connector_PinHeader_2.54mm:PinHeader_1x04_P2.54mm_Vertical
- removed U1: STM32F103C8Tx, Package_QFP:LQFP-48_7x7mm_P0.5mm
- removed U2: AMS1117-3.3, Package_TO_SOT_SMD:SOT-223-3_TabPin2
- removed Y1: Crystal_GND24, Crystal:Crystal_SMD_3225-4Pin_3.2x2.5mm
- added H5: MountingHole, MountingHole:MountingHole_3.2mm_M3, F.Cu at (-14.2, 164.0)
- added H6: MountingHole, MountingHole:MountingHole_3.2mm_M3, F.Cu at (-52.3, 207.5)
- added H7: MountingHole, MountingHole:MountingHole_3.2mm_M3, F.Cu at (-52.3, 215.5)
- added H8: MountingHole, MountingHole:MountingHole_3.2mm_M3, F.Cu at (34.2, 387.5)
- added J1: Conn_01x03_Pin, Connector_PinHeader_2.54mm:PinHeader_1x03_P2.54mm_Vertical, F.Cu at (-109.2, 270.7)
- C1, C6: value 10p -> 220n
- C10, C11: value 1u -> 220n
- C100, C101, C102, C103, C104, C105, C106, C107, C108, C109, C110, C15, C16, C17, C18, C19, C20, C21, C22, C23, C24, C25, C26, C27, C28, C29, C30, C31, C32, C33, C34, C35, C36, C37, C38, C39, C40, C41, C42, C43, C44, C45, C46, C47, C48, C49, C50, C51, C52, C53, C54, C55, C56, C57, C58, C59, C60, C61, C62, C63, C64, C65, C66, C67, C68, C69, C70, C71, C72, C73, C74, C75, C76, C77, C78, C79, C80, C81, C82, C83, C84, C85, C86, C87, C88, C89, C90, C91, C92, C93, C94, C95, C96, C97, C98, C99: moved to F.Cu
- C12, C13: value 22u -> 220n; footprint Capacitor_SMD:C_0805_2012Metric -> Capacitor_SMD:C_0402_1005Metric
- C2: value 10u -> 220n; footprint Capacitor_SMD:C_0603_1608Metric -> Capacitor_SMD:C_0402_1005Metric
- C3, C4, C5, C7, C8: value 100n -> 220n
- C9: value 10n -> 220n
- D1: value LED -> WS2812B; footprint LED_SMD:LED_0603_1608Metric -> LED_SMD:LED_WS2812B_PLCC4_5.0x5.0mm_P3.2mm
- D10, D100, D101, D102, D103, D104, D105, D106, D107, D108, D109, D11, D110, D12, D13, D14, D15, D16, D17, D18, D19, D2, D20, D21, D22, D23, D24, D25, D26, D27, D28, D29, D3, D30, D31, D32, D33, D34, D35, D36, D37, D38, D39, D4, D40, D41, D42, D43, D44, D45, D46, D47, D48, D49, D5, D50, D51, D52, D53, D54, D55, D56, D57, D58, D59, D6, D60, D61, D62, D63, D64, D65, D66, D67, D68, D69, D7, D70, D71, D72, D73, D74, D75, D76, D77, D78, D79, D8, D80, D81, D82, D83, D84, D85, D86, D87, D88, D89, D9, D90, D91, D92, D93, D94, D95, D96, D97, D98, D99: value SK6805 -> WS2812B; footprint LED_SMD:LED_SK6805_PLCC4_2.4x2.7mm_P1.3mm -> LED_SMD:LED_WS2812B_PLCC4_5.0x5.0mm_P3.2mm; moved to F.Cu
- H1, H2, H3, H4: footprint MountingHole:MountingHole_3.2mm_M3 -> MountingHole:MountingHole_2.2mm_M2
- moved H3 562.3 mm to (-114.5, 283.3)
- moved C24 521.2 mm to (-136.1, 285.2)
- moved D12 516.4 mm to (-127.8, 198.9)
- moved H4 514.5 mm to (-114.5, 289.2)
- moved C16 509.2 mm to (-136.1, 269.4)
- moved D13 505.5 mm to (-127.8, 205.5)
- moved C35 503.0 mm to (-133.3, 279.2)
- moved C17 502.4 mm to (-136.1, 271.4)
- moved C22 499.0 mm to (-136.1, 281.2)
- moved C34 497.9 mm to (-133.3, 277.3)
- moved C42 496.6 mm to (-133.3, 293.0)
- moved C63 496.6 mm to (-127.5, 279.2)
- moved C107 486.9 mm to (-118.9, 283.2)
- moved D34 483.2 mm to (-111.0, 198.9)
- moved C18 480.7 mm to (-136.1, 273.3)
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Connections:
- C1 pad 1: /HSE_IN -> VBUS
- C10 pad 1: +3.3VA -> VBUS
- C11 pad 1: +3V3 -> VBUS
- C13 pad 1: +3V3 -> VBUS
- C2 pad 1: +3V3 -> VBUS
- C3 pad 1: +3V3 -> VBUS
- C4 pad 1: +3V3 -> VBUS
- C5 pad 1: /NRST -> VBUS
- C6 pad 1: /HSE_OUT -> VBUS
- C7 pad 1: +3V3 -> VBUS
- C8 pad 1: +3V3 -> VBUS
- C9 pad 1: +3.3VA -> VBUS
- D1 pad 1: Net-(D1-Pad1) -> VBUS
- D1 pad 2: +3V3 -> Net-(D1-DOUT)
- D10 pad 1: Net-(D10-Pad1) -> VBUS
- D10 pad 2: VBUS -> Net-(D1-DIN)
- D10 pad 3: Net-(D10-Pad3) -> GND
- D10 pad 4: GND -> Net-(D10-DIN)
- D100 pad 1: Net-(D100-Pad1) -> VBUS
- D100 pad 2: VBUS -> Net-(D100-DOUT)
- D100 pad 3: Net-(D100-Pad3) -> GND
- D100 pad 4: GND -> Net-(D100-DIN)
- D101 pad 1: Net-(D101-Pad1) -> VBUS
- D101 pad 2: VBUS -> Net-(D101-DOUT)
- D101 pad 3: Net-(D100-Pad1) -> GND
- D101 pad 4: GND -> Net-(D100-DOUT)
- D102 pad 1: Net-(D102-Pad1) -> VBUS
- D102 pad 2: VBUS -> Net-(D102-DOUT)
- D102 pad 3: Net-(D101-Pad1) -> GND
- D102 pad 4: GND -> Net-(D101-DOUT)
- D103 pad 1: Net-(D103-Pad1) -> VBUS
- D103 pad 2: VBUS -> Net-(D103-DOUT)
- D103 pad 3: Net-(D102-Pad1) -> GND
- D103 pad 4: GND -> Net-(D102-DOUT)
- D104 pad 1: Net-(D104-Pad1) -> VBUS
- D104 pad 2: VBUS -> Net-(D104-DOUT)
- D104 pad 3: Net-(D103-Pad1) -> GND
- D104 pad 4: GND -> Net-(D103-DOUT)
- D105 pad 1: Net-(D105-Pad1) -> VBUS
- D105 pad 2: VBUS -> Net-(D105-DOUT)
- D105 pad 3: Net-(D104-Pad1) -> GND
- D105 pad 4: GND -> Net-(D104-DOUT)
- D106 pad 1: Net-(D106-Pad1) -> VBUS
- D106 pad 2: VBUS -> Net-(D106-DOUT)
- D106 pad 3: Net-(D105-Pad1) -> GND
- D106 pad 4: GND -> Net-(D105-DOUT)
- D107 pad 1: Net-(D107-Pad1) -> VBUS
- D107 pad 2: VBUS -> Net-(D107-DOUT)
- D107 pad 3: Net-(D106-Pad1) -> GND
- D107 pad 4: GND -> Net-(D106-DOUT)
- D108 pad 1: Net-(D108-Pad1) -> VBUS
- D108 pad 2: VBUS -> Net-(D108-DOUT)
- D108 pad 3: Net-(D107-Pad1) -> GND
- D108 pad 4: GND -> Net-(D107-DOUT)
- D109 pad 1: Net-(D109-Pad1) -> VBUS
- D109 pad 2: VBUS -> Net-(D109-DOUT)
- D109 pad 3: Net-(D108-Pad1) -> GND
- D109 pad 4: GND -> Net-(D108-DOUT)
- D11 pad 1: Net-(D11-Pad1) -> VBUS
- D11 pad 2: VBUS -> Net-(D10-DIN)
- D11 pad 3: Net-(D10-Pad1) -> GND
- D11 pad 4: GND -> Net-(D11-DIN)
- D110 pad 1: Net-(D110-Pad1) -> VBUS
- D110 pad 2: VBUS -> Net-(D110-DOUT)
- D110 pad 3: Net-(D109-Pad1) -> GND
- D110 pad 4: GND -> Net-(D109-DOUT)
- D12 pad 1: Net-(D12-Pad1) -> VBUS
- D12 pad 2: VBUS -> Net-(D12-DOUT)
- D12 pad 3: Net-(D11-Pad1) -> GND
- D12 pad 4: GND -> Net-(D12-DIN)
- D13 pad 1: Net-(D13-Pad1) -> VBUS
- D13 pad 2: VBUS -> Net-(D13-DOUT)
- D13 pad 3: Net-(D12-Pad1) -> GND
- D13 pad 4: GND -> Net-(D12-DOUT)
- D14 pad 1: Net-(D14-Pad1) -> VBUS
- D14 pad 2: VBUS -> Net-(D14-DOUT)
- D14 pad 3: Net-(D13-Pad1) -> GND
- D14 pad 4: GND -> Net-(D13-DOUT)
- D15 pad 1: Net-(D15-Pad1) -> VBUS
- D15 pad 2: VBUS -> Net-(D15-DOUT)
- D15 pad 3: Net-(D14-Pad1) -> GND
- D15 pad 4: GND -> Net-(D14-DOUT)
- D16 pad 1: Net-(D16-Pad1) -> VBUS
- D16 pad 2: VBUS -> Net-(D16-DOUT)
- D16 pad 3: Net-(D15-Pad1) -> GND
- D16 pad 4: GND -> Net-(D15-DOUT)
- D17 pad 1: Net-(D17-Pad1) -> VBUS
- D17 pad 2: VBUS -> Net-(D17-DOUT)
- D17 pad 3: Net-(D16-Pad1) -> GND
- D17 pad 4: GND -> Net-(D16-DOUT)
- D18 pad 1: Net-(D18-Pad1) -> VBUS
- D18 pad 2: VBUS -> Net-(D18-DOUT)
- D18 pad 3: Net-(D17-Pad1) -> GND
- D18 pad 4: GND -> Net-(D17-DOUT)
- D19 pad 1: Net-(D19-Pad1) -> VBUS
- D19 pad 2: VBUS -> Net-(D19-DOUT)
- D19 pad 3: Net-(D18-Pad1) -> GND
- D19 pad 4: GND -> Net-(D18-DOUT)
- D2 pad 1: Net-(D2-Pad1) -> VBUS
- D2 pad 2: VBUS -> Net-(D2-DOUT)
- D2 pad 3: /LED -> GND
- D2 pad 4: GND -> Net-(D1-DOUT)
- D20 pad 1: Net-(D20-Pad1) -> VBUS
- D20 pad 2: VBUS -> Net-(D20-DOUT)
- D20 pad 3: Net-(D19-Pad1) -> GND
- D20 pad 4: GND -> Net-(D19-DOUT)
- D21 pad 1: Net-(D21-Pad1) -> VBUS
- D21 pad 2: VBUS -> Net-(D21-DOUT)
- D21 pad 3: Net-(D20-Pad1) -> GND
- D21 pad 4: GND -> Net-(D20-DOUT)
- D22 pad 1: Net-(D22-Pad1) -> VBUS
- D22 pad 2: VBUS -> Net-(D22-DOUT)
- D22 pad 3: Net-(D21-Pad1) -> GND
- D22 pad 4: GND -> Net-(D21-DOUT)
- D23 pad 1: Net-(D23-Pad1) -> VBUS
- D23 pad 2: VBUS -> Net-(D23-DOUT)
- D23 pad 3: Net-(D22-Pad1) -> GND
- D23 pad 4: GND -> Net-(D22-DOUT)
- D24 pad 1: Net-(D24-Pad1) -> VBUS
- D24 pad 2: VBUS -> Net-(D24-DOUT)
- D24 pad 3: Net-(D23-Pad1) -> GND
- D24 pad 4: GND -> Net-(D23-DOUT)
- D25 pad 1: Net-(D25-Pad1) -> VBUS
- D25 pad 2: VBUS -> Net-(D25-DOUT)
- D25 pad 3: Net-(D24-Pad1) -> GND
- D25 pad 4: GND -> Net-(D24-DOUT)
- D26 pad 1: Net-(D26-Pad1) -> VBUS
- D26 pad 2: VBUS -> Net-(D26-DOUT)
- D26 pad 3: Net-(D25-Pad1) -> GND
- D26 pad 4: GND -> Net-(D25-DOUT)
- D27 pad 1: Net-(D27-Pad1) -> VBUS
- D27 pad 2: VBUS -> Net-(D27-DOUT)
- D27 pad 3: Net-(D26-Pad1) -> GND
- D27 pad 4: GND -> Net-(D26-DOUT)
- D28 pad 1: Net-(D28-Pad1) -> VBUS
- D28 pad 2: VBUS -> Net-(D28-DOUT)
- D28 pad 3: Net-(D27-Pad1) -> GND
- D28 pad 4: GND -> Net-(D27-DOUT)
- D29 pad 1: Net-(D29-Pad1) -> VBUS
- D29 pad 2: VBUS -> Net-(D29-DOUT)
- D29 pad 3: Net-(D28-Pad1) -> GND
- D29 pad 4: GND -> Net-(D28-DOUT)
- D3 pad 1: Net-(D3-Pad1) -> VBUS
- D3 pad 2: VBUS -> Net-(D3-DOUT)
- D3 pad 3: Net-(D2-Pad1) -> GND
- D3 pad 4: GND -> Net-(D2-DOUT)
- D30 pad 1: Net-(D30-Pad1) -> VBUS
- D30 pad 2: VBUS -> Net-(D30-DOUT)
- D30 pad 3: Net-(D29-Pad1) -> GND
- D30 pad 4: GND -> Net-(D29-DOUT)
- D31 pad 1: Net-(D31-Pad1) -> VBUS
- D31 pad 2: VBUS -> Net-(D31-DOUT)
- D31 pad 3: Net-(D30-Pad1) -> GND
- D31 pad 4: GND -> Net-(D30-DOUT)
- D32 pad 1: Net-(D32-Pad1) -> VBUS
- D32 pad 2: VBUS -> Net-(D32-DOUT)
- D32 pad 3: Net-(D31-Pad1) -> GND
- D32 pad 4: GND -> Net-(D31-DOUT)
- D33 pad 1: Net-(D33-Pad1) -> VBUS
- D33 pad 2: VBUS -> Net-(D33-DOUT)
- D33 pad 3: Net-(D32-Pad1) -> GND
- D33 pad 4: GND -> Net-(D32-DOUT)
- D34 pad 1: Net-(D34-Pad1) -> VBUS
- D34 pad 2: VBUS -> Net-(D34-DOUT)
- D34 pad 3: Net-(D33-Pad1) -> GND
- D34 pad 4: GND -> Net-(D33-DOUT)
- D35 pad 1: Net-(D35-Pad1) -> VBUS
- D35 pad 2: VBUS -> Net-(D35-DOUT)
- D35 pad 3: Net-(D34-Pad1) -> GND
- D35 pad 4: GND -> Net-(D34-DOUT)
- D36 pad 1: Net-(D36-Pad1) -> VBUS
- D36 pad 2: VBUS -> Net-(D36-DOUT)
- D36 pad 3: Net-(D35-Pad1) -> GND
- D36 pad 4: GND -> Net-(D35-DOUT)
- D37 pad 1: Net-(D37-Pad1) -> VBUS
- D37 pad 2: VBUS -> Net-(D37-DOUT)
- D37 pad 3: Net-(D36-Pad1) -> GND
- D37 pad 4: GND -> Net-(D36-DOUT)
- D38 pad 1: Net-(D38-Pad1) -> VBUS
- D38 pad 2: VBUS -> Net-(D38-DOUT)
- D38 pad 3: Net-(D37-Pad1) -> GND
- D38 pad 4: GND -> Net-(D37-DOUT)
- D39 pad 1: Net-(D39-Pad1) -> VBUS
- D39 pad 2: VBUS -> Net-(D39-DOUT)
- D39 pad 3: Net-(D38-Pad1) -> GND
- D39 pad 4: GND -> Net-(D38-DOUT)
- D4 pad 1: Net-(D4-Pad1) -> VBUS
- D4 pad 2: VBUS -> Net-(D4-DOUT)
- D4 pad 3: Net-(D3-Pad1) -> GND
- D4 pad 4: GND -> Net-(D3-DOUT)
- D40 pad 1: Net-(D40-Pad1) -> VBUS
- D40 pad 2: VBUS -> Net-(D40-DOUT)
- D40 pad 3: Net-(D39-Pad1) -> GND
- D40 pad 4: GND -> Net-(D39-DOUT)
- D41 pad 1: Net-(D41-Pad1) -> VBUS
- D41 pad 2: VBUS -> Net-(D41-DOUT)
- D41 pad 3: Net-(D40-Pad1) -> GND
- D41 pad 4: GND -> Net-(D40-DOUT)
- D42 pad 1: Net-(D42-Pad1) -> VBUS
- D42 pad 2: VBUS -> Net-(D42-DOUT)
- D42 pad 3: Net-(D41-Pad1) -> GND
- D42 pad 4: GND -> Net-(D41-DOUT)
- D43 pad 1: Net-(D43-Pad1) -> VBUS
- D43 pad 2: VBUS -> Net-(D43-DOUT)
- D43 pad 3: Net-(D42-Pad1) -> GND
- D43 pad 4: GND -> Net-(D42-DOUT)
- D44 pad 1: Net-(D44-Pad1) -> VBUS
- D44 pad 2: VBUS -> Net-(D44-DOUT)
- D44 pad 3: Net-(D43-Pad1) -> GND
- D44 pad 4: GND -> Net-(D43-DOUT)
- D45 pad 1: Net-(D45-Pad1) -> VBUS
- D45 pad 2: VBUS -> Net-(D45-DOUT)
- D45 pad 3: Net-(D44-Pad1) -> GND
- D45 pad 4: GND -> Net-(D44-DOUT)
- D46 pad 1: Net-(D46-Pad1) -> VBUS
- D46 pad 2: VBUS -> Net-(D46-DOUT)
- D46 pad 3: Net-(D45-Pad1) -> GND
- D46 pad 4: GND -> Net-(D45-DOUT)
- D47 pad 1: Net-(D47-Pad1) -> VBUS
- D47 pad 2: VBUS -> Net-(D47-DOUT)
- D47 pad 3: Net-(D46-Pad1) -> GND
- D47 pad 4: GND -> Net-(D46-DOUT)
- D48 pad 1: Net-(D48-Pad1) -> VBUS
- D48 pad 2: VBUS -> Net-(D48-DOUT)
- D48 pad 3: Net-(D47-Pad1) -> GND
- D48 pad 4: GND -> Net-(D47-DOUT)
- D49 pad 1: Net-(D49-Pad1) -> VBUS
- D49 pad 2: VBUS -> Net-(D49-DOUT)
- D49 pad 3: Net-(D48-Pad1) -> GND
- D49 pad 4: GND -> Net-(D48-DOUT)
- D5 pad 1: Net-(D5-Pad1) -> VBUS
- D5 pad 2: VBUS -> Net-(D5-DOUT)
- D5 pad 3: Net-(D4-Pad1) -> GND
- D5 pad 4: GND -> Net-(D4-DOUT)
- D50 pad 1: Net-(D50-Pad1) -> VBUS
- D50 pad 2: VBUS -> Net-(D50-DOUT)
- D50 pad 3: Net-(D49-Pad1) -> GND
- D50 pad 4: GND -> Net-(D49-DOUT)
- D51 pad 1: Net-(D51-Pad1) -> VBUS
- D51 pad 2: VBUS -> Net-(D51-DOUT)
- D51 pad 3: Net-(D50-Pad1) -> GND
- D51 pad 4: GND -> Net-(D50-DOUT)
- D52 pad 1: Net-(D52-Pad1) -> VBUS
- D52 pad 2: VBUS -> Net-(D52-DOUT)
- D52 pad 3: Net-(D51-Pad1) -> GND
- D52 pad 4: GND -> Net-(D51-DOUT)
- D53 pad 1: Net-(D53-Pad1) -> VBUS
- D53 pad 2: VBUS -> Net-(D53-DOUT)
- D53 pad 3: Net-(D52-Pad1) -> GND
- D53 pad 4: GND -> Net-(D52-DOUT)
- D54 pad 1: Net-(D54-Pad1) -> VBUS
- D54 pad 2: VBUS -> Net-(D54-DOUT)
- D54 pad 3: Net-(D53-Pad1) -> GND
- D54 pad 4: GND -> Net-(D53-DOUT)
- D55 pad 1: Net-(D55-Pad1) -> VBUS
- D55 pad 2: VBUS -> Net-(D100-DIN)
- D55 pad 3: Net-(D54-Pad1) -> GND
- D55 pad 4: GND -> Net-(D54-DOUT)
- D56 pad 1: Net-(D56-Pad1) -> VBUS
- D56 pad 2: VBUS -> Net-(D56-DOUT)
- D56 pad 3: Net-(D55-Pad1) -> GND
- D56 pad 4: GND -> Net-(D56-DIN)
- D57 pad 1: Net-(D57-Pad1) -> VBUS
- D57 pad 2: VBUS -> Net-(D57-DOUT)
- D57 pad 3: Net-(D56-Pad1) -> GND
- D57 pad 4: GND -> Net-(D56-DOUT)
- D58 pad 1: Net-(D58-Pad1) -> VBUS
- D58 pad 2: VBUS -> Net-(D58-DOUT)
- D58 pad 3: Net-(D57-Pad1) -> GND
- D58 pad 4: GND -> Net-(D57-DOUT)
- D59 pad 1: Net-(D59-Pad1) -> VBUS
- D59 pad 2: VBUS -> Net-(D59-DOUT)
- D59 pad 3: Net-(D58-Pad1) -> GND
- D59 pad 4: GND -> Net-(D58-DOUT)
- D6 pad 1: Net-(D6-Pad1) -> VBUS
- D6 pad 2: VBUS -> Net-(D6-DOUT)
- D6 pad 3: Net-(D5-Pad1) -> GND
- D6 pad 4: GND -> Net-(D5-DOUT)
- D60 pad 1: Net-(D60-Pad1) -> VBUS
- D60 pad 2: VBUS -> Net-(D60-DOUT)
- D60 pad 3: Net-(D59-Pad1) -> GND
- D60 pad 4: GND -> Net-(D59-DOUT)
- D61 pad 1: Net-(D61-Pad1) -> VBUS
- D61 pad 2: VBUS -> Net-(D61-DOUT)
- D61 pad 3: Net-(D60-Pad1) -> GND
- D61 pad 4: GND -> Net-(D60-DOUT)
- D62 pad 1: Net-(D62-Pad1) -> VBUS
- D62 pad 2: VBUS -> Net-(D62-DOUT)
- D62 pad 3: Net-(D61-Pad1) -> GND
- D62 pad 4: GND -> Net-(D61-DOUT)
- D63 pad 1: Net-(D63-Pad1) -> VBUS
- D63 pad 2: VBUS -> Net-(D63-DOUT)
- D63 pad 3: Net-(D62-Pad1) -> GND
- D63 pad 4: GND -> Net-(D62-DOUT)
- D64 pad 1: Net-(D64-Pad1) -> VBUS
- D64 pad 2: VBUS -> Net-(D64-DOUT)
- D64 pad 3: Net-(D63-Pad1) -> GND
- D64 pad 4: GND -> Net-(D63-DOUT)
- D65 pad 1: Net-(D65-Pad1) -> VBUS
- D65 pad 2: VBUS -> Net-(D65-DOUT)
- D65 pad 3: Net-(D64-Pad1) -> GND
- D65 pad 4: GND -> Net-(D64-DOUT)
- D66 pad 1: Net-(D66-Pad1) -> VBUS
- D66 pad 2: VBUS -> unconnected-(D66-DOUT-Pad2)
- D66 pad 3: Net-(D65-Pad1) -> GND
- D66 pad 4: GND -> Net-(D65-DOUT)
- D67 pad 1: Net-(D67-Pad1) -> VBUS
- D67 pad 2: VBUS -> Net-(D56-DIN)
- D67 pad 3: Net-(D66-Pad1) -> GND
- D67 pad 4: GND -> Net-(D67-DIN)
- D68 pad 1: Net-(D68-Pad1) -> VBUS
- D68 pad 2: VBUS -> Net-(D67-DIN)
- D68 pad 3: Net-(D67-Pad1) -> GND
- D68 pad 4: GND -> Net-(D68-DIN)
- D69 pad 1: Net-(D69-Pad1) -> VBUS
- D69 pad 2: VBUS -> Net-(D68-DIN)
- D69 pad 3: Net-(D68-Pad1) -> GND
- D69 pad 4: GND -> Net-(D69-DIN)
- D7 pad 1: Net-(D7-Pad1) -> VBUS
- D7 pad 2: VBUS -> Net-(D7-DOUT)
- D7 pad 3: Net-(D6-Pad1) -> GND
- D7 pad 4: GND -> Net-(D6-DOUT)
- D70 pad 1: Net-(D70-Pad1) -> VBUS
- D70 pad 2: VBUS -> Net-(D69-DIN)
- D70 pad 3: Net-(D69-Pad1) -> GND
- D70 pad 4: GND -> Net-(D70-DIN)
- D71 pad 1: Net-(D71-Pad1) -> VBUS
- D71 pad 2: VBUS -> Net-(D70-DIN)
- D71 pad 3: Net-(D70-Pad1) -> GND
- D71 pad 4: GND -> Net-(D71-DIN)
- D72 pad 1: Net-(D72-Pad1) -> VBUS
- D72 pad 2: VBUS -> Net-(D71-DIN)
- D72 pad 3: Net-(D71-Pad1) -> GND
- D72 pad 4: GND -> Net-(D72-DIN)
- D73 pad 1: Net-(D73-Pad1) -> VBUS
- D73 pad 2: VBUS -> Net-(D72-DIN)
- D73 pad 3: Net-(D72-Pad1) -> GND
- D73 pad 4: GND -> Net-(D73-DIN)
- D74 pad 1: Net-(D74-Pad1) -> VBUS
- D74 pad 2: VBUS -> Net-(D73-DIN)
- D74 pad 3: Net-(D73-Pad1) -> GND
- D74 pad 4: GND -> Net-(D74-DIN)
- D75 pad 1: Net-(D75-Pad1) -> VBUS
- D75 pad 2: VBUS -> Net-(D74-DIN)
- D75 pad 3: Net-(D74-Pad1) -> GND
- D75 pad 4: GND -> Net-(D75-DIN)
- D76 pad 1: Net-(D76-Pad1) -> VBUS
- D76 pad 2: VBUS -> Net-(D75-DIN)
- D76 pad 3: Net-(D75-Pad1) -> GND
- D76 pad 4: GND -> Net-(D76-DIN)
- D77 pad 1: Net-(D77-Pad1) -> VBUS
- D77 pad 2: VBUS -> Net-(D76-DIN)
- D77 pad 3: Net-(D76-Pad1) -> GND
- D77 pad 4: GND -> Net-(D77-DIN)
- D78 pad 1: Net-(D78-Pad1) -> VBUS
- D78 pad 2: VBUS -> Net-(D78-DOUT)
- D78 pad 3: Net-(D77-Pad1) -> GND
- D78 pad 4: GND -> Net-(D78-DIN)
- D79 pad 1: Net-(D79-Pad1) -> VBUS
- D79 pad 2: VBUS -> Net-(D79-DOUT)
- D79 pad 3: Net-(D78-Pad1) -> GND
- D79 pad 4: GND -> Net-(D78-DOUT)
- D8 pad 1: Net-(D8-Pad1) -> VBUS
- D8 pad 2: VBUS -> Net-(D8-DOUT)
- D8 pad 3: Net-(D7-Pad1) -> GND
- D8 pad 4: GND -> Net-(D7-DOUT)
- D80 pad 1: Net-(D80-Pad1) -> VBUS
- D80 pad 2: VBUS -> Net-(D80-DOUT)
- D80 pad 3: Net-(D79-Pad1) -> GND
- D80 pad 4: GND -> Net-(D79-DOUT)
- D81 pad 1: Net-(D81-Pad1) -> VBUS
- D81 pad 2: VBUS -> Net-(D81-DOUT)
- D81 pad 3: Net-(D80-Pad1) -> GND
- D81 pad 4: GND -> Net-(D80-DOUT)
- D82 pad 1: Net-(D82-Pad1) -> VBUS
- D82 pad 2: VBUS -> Net-(D82-DOUT)
- D82 pad 3: Net-(D81-Pad1) -> GND
- D82 pad 4: GND -> Net-(D81-DOUT)
- D83 pad 1: Net-(D83-Pad1) -> VBUS
- D83 pad 2: VBUS -> Net-(D83-DOUT)
- D83 pad 3: Net-(D82-Pad1) -> GND
- D83 pad 4: GND -> Net-(D82-DOUT)
- D84 pad 1: Net-(D84-Pad1) -> VBUS
- D84 pad 2: VBUS -> Net-(D84-DOUT)
- D84 pad 3: Net-(D83-Pad1) -> GND
- D84 pad 4: GND -> Net-(D83-DOUT)
- D85 pad 1: Net-(D85-Pad1) -> VBUS
- D85 pad 2: VBUS -> Net-(D85-DOUT)
- D85 pad 3: Net-(D84-Pad1) -> GND
- D85 pad 4: GND -> Net-(D84-DOUT)
- D86 pad 1: Net-(D86-Pad1) -> VBUS
- D86 pad 2: VBUS -> Net-(D86-DOUT)
- D86 pad 3: Net-(D85-Pad1) -> GND
- D86 pad 4: GND -> Net-(D85-DOUT)
- D87 pad 1: Net-(D87-Pad1) -> VBUS
- D87 pad 2: VBUS -> Net-(D87-DOUT)
- D87 pad 3: Net-(D86-Pad1) -> GND
- D87 pad 4: GND -> Net-(D86-DOUT)
- D88 pad 1: Net-(D88-Pad1) -> VBUS
- D88 pad 2: VBUS -> Net-(D77-DIN)
- D88 pad 3: Net-(D87-Pad1) -> GND
- D88 pad 4: GND -> Net-(D87-DOUT)
- D89 pad 1: Net-(D89-Pad1) -> VBUS
- D89 pad 2: VBUS -> Net-(D78-DIN)
- D89 pad 3: Net-(D88-Pad1) -> GND
- D89 pad 4: GND -> Net-(D89-DIN)
- D9 pad 1: Net-(D10-Pad3) -> VBUS
- D9 pad 2: VBUS -> Net-(D12-DIN)
- D9 pad 3: Net-(D8-Pad1) -> GND
- D9 pad 4: GND -> Net-(D8-DOUT)
- D90 pad 1: Net-(D90-Pad1) -> VBUS
- D90 pad 2: VBUS -> Net-(D89-DIN)
- D90 pad 3: Net-(D89-Pad1) -> GND
- D90 pad 4: GND -> Net-(D90-DIN)
- D91 pad 1: Net-(D91-Pad1) -> VBUS
- D91 pad 2: VBUS -> Net-(D90-DIN)
- D91 pad 3: Net-(D90-Pad1) -> GND
- D91 pad 4: GND -> Net-(D91-DIN)
- D92 pad 1: Net-(D92-Pad1) -> VBUS
- D92 pad 2: VBUS -> Net-(D91-DIN)
- D92 pad 3: Net-(D91-Pad1) -> GND
- D92 pad 4: GND -> Net-(D92-DIN)
- D93 pad 1: Net-(D93-Pad1) -> VBUS
- D93 pad 2: VBUS -> Net-(D92-DIN)
- D93 pad 3: Net-(D92-Pad1) -> GND
- D93 pad 4: GND -> Net-(D93-DIN)
- D94 pad 1: Net-(D94-Pad1) -> VBUS
- D94 pad 2: VBUS -> Net-(D93-DIN)
- D94 pad 3: Net-(D93-Pad1) -> GND
- D94 pad 4: GND -> Net-(D94-DIN)
- D95 pad 1: Net-(D95-Pad1) -> VBUS
- D95 pad 2: VBUS -> Net-(D94-DIN)
- D95 pad 3: Net-(D94-Pad1) -> GND
- D95 pad 4: GND -> Net-(D95-DIN)
- D96 pad 1: Net-(D96-Pad1) -> VBUS
- D96 pad 2: VBUS -> Net-(D95-DIN)
- D96 pad 3: Net-(D95-Pad1) -> GND
- D96 pad 4: GND -> Net-(D96-DIN)
- D97 pad 1: Net-(D97-Pad1) -> VBUS
- D97 pad 2: VBUS -> Net-(D96-DIN)
- D97 pad 3: Net-(D96-Pad1) -> GND
- D97 pad 4: GND -> Net-(D97-DIN)
- D98 pad 1: Net-(D98-Pad1) -> VBUS
- D98 pad 2: VBUS -> Net-(D97-DIN)
- D98 pad 3: Net-(D97-Pad1) -> GND
- D98 pad 4: GND -> Net-(D98-DIN)
- D99 pad 1: Net-(D100-Pad3) -> VBUS
- D99 pad 2: VBUS -> Net-(D98-DIN)
- D99 pad 3: Net-(D98-Pad1) -> GND
- D99 pad 4: GND -> Net-(D110-DOUT)
Routing:
- net VBUS: track 4281.3 -> 0.00 mm, vias 141 -> 0
- net GND: track 3936.4 -> 0.00 mm, vias 233 -> 0
- net +3V3: track 259.0 -> 0.00 mm, vias 9 -> 0
- net /LED: track 147.4 -> 0.00 mm, vias 3 -> 0
- net /BTN_H: track 73.9 -> 0.00 mm, vias 2 -> 0
- net /I2C2_SCL: track 60.6 -> 0.00 mm, vias 2 -> 0
- net /I2C2_SDA: track 59.9 -> 0.00 mm
- net /BTN_M: track 55.7 -> 0.00 mm, vias 2 -> 0
- net /SWCLK: track 48.0 -> 0.00 mm, vias 2 -> 0
- net /SWDIO: track 44.6 -> 0.00 mm, vias 2 -> 0
- net Net-(D12-Pad1): track 39.2 -> 0.00 mm
- net Net-(D78-Pad1): track 39.2 -> 0.00 mm
- net Net-(D34-Pad1): track 39.2 -> 0.00 mm
- net Net-(D89-Pad1): track 39.2 -> 0.00 mm
- net Net-(D56-Pad1): track 39.2 -> 0.00 mm
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- removed copper zone on B.Cu, net GND
Other:
- net class Default removed
- board text removed: "SDA"
