File: mcu/qclock.kicad_pcb (KiCad board)
At the start: 2 copper layers, 61.2 x 34 mm, 43 parts, among them J1 Conn_01x04_Male, J2 Conn_01x04_Male, J3 USB_B_Micro, J4 Conn_01x04_Male, J5 Conn_01x03_Male, SW1 SW_SPDT, SW2 SW_Push, SW3 SW_Push, SW4 SW_Push, U1 STM32F103C8Tx, U2 AMS1117-3.3, Y1 Crystal_GND24

Commit message: Update mcu
Parts:
- J3: footprint Connector_USB:USB_Micro-B_Wuerth_629105150521 -> footprints:CUS-12TB_NDC
- moved J3 2.65 mm to (171.8, 88.0)
Routing:
- net VBUS: track 104.6 -> 82.7 mm, vias 2 -> 4
- net /USB_D-: track 12.5 -> 14.6 mm
- net /USB_D+: track 12.4 -> 14.6 mm
