File: mcu/qclock.kicad_sch (KiCad schematic)
At the start: 43 parts, among them J1 Conn_01x04_Male, J2 Conn_01x04_Male, J3 USB_B_Micro, J4 Conn_01x04_Male, J5 Conn_01x03_Male, SW1 SW_SPDT, SW2 SW_Push, SW3 SW_Push, SW4 SW_Push, U1 STM32F103C8Tx, U2 AMS1117-3.3, Y1 Crystal_GND24

Commit message: Update mcu
Parts:
- J3: footprint Connector_USB:USB_Micro-B_Wuerth_629105150521 -> footprints:CUS-12TB_NDC; JLCPCB Part #（optional） C879727 -> C40943
Changed lines of the file:
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@@
 			)
 		)
-		(property "Footprint" "Connector_USB:USB_Micro-B_Wuerth_629105150521"
+		(property "Footprint" "footprints:CUS-12TB_NDC"
 			(at 162.56 116.84 0)
 			(effects
@@
 			)
 		)
-		(property "JLCPCB Part #（optional）" " C879727"
+		(property "JLCPCB Part #（optional）" " C40943"
 			(at 166.37 115.57 0)
 			(effects
